Commit message: Loading Gazebo with controllers and working

File: src/erobotics_description/urdf/adaptative_gripper.urdf.xacro (robot description, xacro)
@@ -10,13 +10,13 @@
     </joint>
     <!-- Links del Gripper -->
-    <xacro:m_link_mesh name="gripper_base" mesh_file="gripper_base.dae" origin_xyz="0 0 -0.012" origin_rpy="0 0 0" />
-    <xacro:m_link_mesh name="gripper_left1" mesh_file="gripper_left1.dae" origin_xyz="0.039 -0.0133 -0.012" origin_rpy="0 0 0" />
-    <xacro:m_link_mesh name="gripper_left2" mesh_file="gripper_left2.dae" origin_xyz="0.005 -0.0195 -0.012" origin_rpy="0 0 0" />
-    <xacro:m_link_mesh name="gripper_left3" mesh_file="gripper_left3.dae" origin_xyz="0.012 0.0025 -0.012" origin_rpy="0 0 0" />
-    <xacro:m_link_mesh name="gripper_right1" mesh_file="gripper_right1.dae" origin_xyz="-0.039 -0.0133 -0.012" origin_rpy="0 0 0" />
-    <xacro:m_link_mesh name="gripper_right2" mesh_file="gripper_right2.dae" origin_xyz="-0.005 -0.0195 -0.012" origin_rpy="0 0 0" />
-    <xacro:m_link_mesh name="gripper_right3" mesh_file="gripper_right3.dae" origin_xyz="-0.012 0.0025 -0.012" origin_rpy="0 0 0" />
+    <xacro:m_link_mesh name="gripper_base" mesh_file="gripper_base.dae" origin_xyz="0 0 -0.012" origin_rpy="0 0 0" mass="0.001"/>
+    <xacro:m_link_mesh name="gripper_left1" mesh_file="gripper_left1.dae" origin_xyz="0.039 -0.0133 -0.012" origin_rpy="0 0 0" mass="0.001"/>
+    <xacro:m_link_mesh name="gripper_left2" mesh_file="gripper_left2.dae" origin_xyz="0.005 -0.0195 -0.012" origin_rpy="0 0 0" mass="0.001"/>
+    <xacro:m_link_mesh name="gripper_left3" mesh_file="gripper_left3.dae" origin_xyz="0.012 0.0025 -0.012" origin_rpy="0 0 0" mass="0.001"/>
+    <xacro:m_link_mesh name="gripper_right1" mesh_file="gripper_right1.dae" origin_xyz="-0.039 -0.0133 -0.012" origin_rpy="0 0 0" mass="0.001"/>
+    <xacro:m_link_mesh name="gripper_right2" mesh_file="gripper_right2.dae" origin_xyz="-0.005 -0.0195 -0.012" origin_rpy="0 0 0" mass="0.001"/>
+    <xacro:m_link_mesh name="gripper_right3" mesh_file="gripper_right3.dae" origin_xyz="-0.012 0.0025 -0.012" origin_rpy="0 0 0" mass="0.001"/>
     <!-- Articulaciones internas del Gripper -->
-    <joint name="gripper_controller" type="revolute">
+    <joint name="gripper_controllable_joint" type="revolute">
       <axis xyz="0 0 1"/><limit effort="1000.0" lower="-0.74" upper="0.15" velocity="0"/>
       <parent link="gripper_base"/><child link="gripper_left3"/><origin xyz="-0.012 0.005 0" rpy="0 0 0"/>
@@ -25,33 +25,33 @@
       <axis xyz="0 0 1"/><limit effort="1000.0" lower="-0.8" upper="0.5" velocity="0"/>
       <parent link="gripper_base"/><child link="gripper_left2"/><origin xyz="-0.005 0.027 0" rpy="0 0 0"/>
-      <mimic joint="gripper_controller" multiplier="1.0" offset="0" />
+      <mimic joint="gripper_controllable_joint" multiplier="1.0" offset="0" />
     </joint>
     <joint name="gripper_left3_to_gripper_left1" type="revolute">
       <axis xyz="0 0 1"/><limit effort="1000.0" lower="-0.5" upper="0.5" velocity="0"/>
       <parent link="gripper_left3"/><child link="gripper_left1"/><origin xyz="-0.027 0.016 0" rpy="0 0 0"/>
-      <mimic joint="gripper_controller" multiplier="-1.0" offset="0" />
+      <mimic joint="gripper_controllable_joint" multiplier="-1.0" offset="0" />
     </joint>
     <joint name="gripper_base_to_gripper_right3" type="revolute">
       <axis xyz="0 0 1"/><limit effort="1000.0" lower="-0.15" upper="0.7" velocity="0"/>
       <parent link="gripper_base"/><child link="gripper_right3"/><origin xyz="0.012 0.005 0" rpy="0 0 0"/>
-      <mimic joint="gripper_controller" multiplier="-1.0" offset="0" />
+      <mimic joint="gripper_controllable_joint" multiplier="-1.0" offset="0" />
     </joint>
     <joint name="gripper_base_to_gripper_right2" type="revolute">
       <axis xyz="0 0 1"/><limit effort="1000.0" lower="-0.5" upper="0.8" velocity="0"/>
       <parent link="gripper_base"/><child link="gripper_right2"/><origin xyz="0.005 0.027 0" rpy="0 0 0"/>
-      <mimic joint="gripper_controller" multiplier="-1.0" offset="0" />
+      <mimic joint="gripper_controllable_joint" multiplier="-1.0" offset="0" />
     </joint>
     <joint name="gripper_right3_to_gripper_right1" type="revolute">
       <axis xyz="0 0 1"/><limit effort="1000.0" lower="-0.5" upper="0.5" velocity="0"/>
       <parent link="gripper_right3"/><child link="gripper_right1"/><origin xyz="0.027 0.016 0" rpy="0 0 0"/>
-      <mimic joint="gripper_controller" multiplier="1.0" offset="0" />
+      <mimic joint="gripper_controllable_joint" multiplier="1.0" offset="0" />
     </joint>
   <!-- Definición de ros2_control para el Gripper -->
     <!-- Articulación Maestra del Gripper -->
-  <ros2_control name="GazeboSimSystem" type="system">
+  <ros2_control name="GazeboSimSystemGripper" type="system">
     <hardware>
       <plugin>gz_ros2_control/GazeboSimSystem</plugin>
     </hardware>
-      <joint name="gripper_controller">
+      <joint name="gripper_controllable_joint">
         <command_interface name="position"/>
         <state_interface name="position">

File: src/erobotics_description/urdf/mycobot_280_arduino.urdf.xacro (robot description, xacro)
@@ -62,10 +62,10 @@
   <!-- Articulaciones del Brazo -->
   <joint name="g_base_to_joint1" type="fixed"><parent link="g_base"/><child link="joint1"/><origin xyz="0 0 0" rpy="0 0 0"/></joint>
-  <joint name="joint2_to_joint1" type="revolute"><axis xyz="0 0 1"/><limit effort="1000.0" lower="-2.9321" upper="2.9321" velocity="0"/><parent link="joint1"/><child link="joint2"/><origin xyz="0 0 0.13156" rpy="0 0 0"/></joint>
-  <joint name="joint3_to_joint2" type="revolute"><axis xyz="0 0 1"/><limit effort="1000.0" lower="-2.3561" upper="2.3561" velocity="0"/><parent link="joint2"/><child link="joint3"/><origin xyz="0 0 0" rpy="0 1.5708 -1.5708"/></joint>
-  <joint name="joint4_to_joint3" type="revolute"><axis xyz="0 0 1"/><limit effort="1000.0" lower="-2.6179" upper="2.6179" velocity="0"/><parent link="joint3"/><child link="joint4"/><origin xyz="-0.1104 0 0" rpy="0 0 0"/></joint>
-  <joint name="joint5_to_joint4" type="revolute"><axis xyz="0 0 1"/><limit effort="1000.0" lower="-2.5307" upper="2.5307" velocity="0"/><parent link="joint4"/><child link="joint5"/><origin xyz="-0.096 0 0.06462" rpy="0 0 -1.5708"/></joint>
-  <joint name="joint6_to_joint5" type="revolute"><axis xyz="0 0 1"/><limit effort="1000.0" lower="-2.8797" upper="2.8797" velocity="0"/><parent link="joint5"/><child link="joint6"/><origin xyz="0 -0.07318 0" rpy="1.5708 -1.5708 0"/></joint>
-  <joint name="joint6output_to_joint6" type="revolute"><axis xyz="0 0 1"/><limit effort="1000.0" lower="-3.14" upper="3.14159" velocity="0"/><parent link="joint6"/><child link="joint6_flange"/><origin xyz="0 0.0456 0" rpy="-1.5708 0 0"/></joint>
+  <joint name="joint2_to_joint1" type="revolute"><axis xyz="0 0 1"/><limit effort="1000.0" lower="-2.9321" upper="2.9321" velocity="0.3"/><parent link="joint1"/><child link="joint2"/><origin xyz="0 0 0.13156" rpy="0 0 0"/></joint>
+  <joint name="joint3_to_joint2" type="revolute"><axis xyz="0 0 1"/><limit effort="1000.0" lower="-2.3561" upper="2.3561" velocity="0.3"/><parent link="joint2"/><child link="joint3"/><origin xyz="0 0 0" rpy="0 1.5708 -1.5708"/></joint>
+  <joint name="joint4_to_joint3" type="revolute"><axis xyz="0 0 1"/><limit effort="1000.0" lower="-2.6179" upper="2.6179" velocity="0.3"/><parent link="joint3"/><child link="joint4"/><origin xyz="-0.1104 0 0" rpy="0 0 0"/></joint>
+  <joint name="joint5_to_joint4" type="revolute"><axis xyz="0 0 1"/><limit effort="1000.0" lower="-2.5307" upper="2.5307" velocity="0.3"/><parent link="joint4"/><child link="joint5"/><origin xyz="-0.096 0 0.06462" rpy="0 0 -1.5708"/></joint>
+  <joint name="joint6_to_joint5" type="revolute"><axis xyz="0 0 1"/><limit effort="1000.0" lower="-2.8797" upper="2.8797" velocity="0.3"/><parent link="joint5"/><child link="joint6"/><origin xyz="0 -0.07318 0" rpy="1.5708 -1.5708 0"/></joint>
+  <joint name="joint6output_to_joint6" type="revolute"><axis xyz="0 0 1"/><limit effort="1000.0" lower="-3.14" upper="3.14159" velocity="0.3"/><parent link="joint6"/><child link="joint6_flange"/><origin xyz="0 0.0456 0" rpy="-1.5708 0 0"/></joint>
   <!-- LLAMADA CONDICIONAL: Carga la pinza si use_gripper es true -->
   <xacro:if value="$(arg use_gripper)">
