Commit message: mycobot_280 working in gazebo +  moveit

File: src/erobotics_description/urdf/mycobot_280_arduino.urdf.xacro (robot description, xacro)
@@ -7,5 +7,5 @@
   <xacro:property name="mesh_path" value="package://erobotics_description/meshes" />
   <xacro:property name="width" value=".2" />
-  <xacro:property name="default_mass" value="0.1" />
+  <xacro:property name="default_mass" value="0.01" />
   <!-- Incluir configuración de Gazebo y el archivo de la Pinza -->
   <xacro:include filename="erobotics_ros2_control.xacro" />

File: src/erobotics_description/urdf/rgb_camera.xacro (robot description, xacro)
@@ -22,5 +22,5 @@
       </collision>
       <inertial>
-        <mass value="0.1"/>
+        <mass value="0.01"/>
         <inertia ixx="0.0001" ixy="0" ixz="0" iyy="0.0001" iyz="0" izz="0.0001"/>
       </inertial>
